File: pcb/choc/bgkeeb.kicad_pcb (KiCad board)
At the start: 2 copper layers, 98.4 x 90.5 mm, 106 parts, among them J1 Pimoroni, SW1 SW_Push, SW11 SW_Push, SW12 SW_Push, SW13 SW_Push, SW14 SW_Push, SW15 SW_Push, SW2 SW_Push, SW21 SW_Push, SW22 SW_Push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

Commit message: choc bgkeeb is complete
Routing:
- net row3: track 0.00 -> 175.4 mm, vias 1 -> 12
- net col4: track 0.00 -> 135.1 mm, vias 0 -> 1
- net col0: track 0.00 -> 131.7 mm, vias 0 -> 4
- net row2: track 0.00 -> 122.6 mm, vias 0 -> 8
- net col2: track 0.00 -> 121.5 mm, vias 0 -> 4
- net col3: track 0.00 -> 113.1 mm, vias 0 -> 1
- net col1: track 0.00 -> 97.7 mm, vias 0 -> 1
- net sda: track 0.00 -> 87.8 mm, vias 0 -> 8
- net row0: track 0.00 -> 84.9 mm, vias 1 -> 8
- net scl: track 0.00 -> 77.2 mm, vias 0 -> 1
- net GND: track 692.4 -> 632.1 mm, vias 61 -> 54
- net Net-(D51-Pad2): track 0.00 -> 25.6 mm, vias 0 -> 4
- net Net-(D39-Pad2): track 0.00 -> 22.3 mm
- net Net-(D30-Pad2): track 0.00 -> 10.2 mm, vias 0 -> 1
- net Net-(D14-Pad2): track 0.00 -> 10.2 mm, vias 0 -> 1
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